File: pcb/StickerCutter.kicad_sch (KiCad schematic)
At the start: 18 parts, among them J1 24V, J3 Line Sensor, J4 Paper Sensor, J5 ENC_0, J6 ENC_1, SW1 F1, SW2 F2, SW3 Forward, SW4 Backward, SW5 Left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

Commit message: Added buttons, improved manual mode
Parts:
- SW3: value Forward -> In
- SW4: value Backward -> Out
Connections:
- net Backward: no longer U1.1 (GPIO0)
- net Forward: no longer U1.6 (GPIO4)
- new net In: U1.6 (GPIO4)
- new net Out: U1.1 (GPIO0)
Changed lines of the file:
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@@
     (effects (font (size 1.27 1.27)) (justify left bottom))
   )
-  (label "Forward" (at 40.64 106.68 0)
+  (label "In" (at 40.64 106.68 0)
     (effects (font (size 1.27 1.27)) (justify left bottom))
   )
@@
     (effects (font (size 1.27 1.27)) (justify left bottom))
   )
-  (label "Backward" (at 40.64 93.98 0)
+  (label "Out" (at 40.64 93.98 0)
     (effects (font (size 1.27 1.27)) (justify left bottom))
   )
@@
     (in_bom yes) (on_board yes) (fields_autoplaced)
     (property "Reference" "SW3" (id 0) (at 119.38 171.45 0))
-    (property "Value" "Forward" (id 1) (at 119.38 173.99 0))
+    (property "Value" "In" (id 1) (at 119.38 173.99 0))
     (property "Footprint" "Button_Switch_THT:SW_PUSH_6mm" (id 2) (at 119.38 173.99 0)
       (effects (font (size 1.27 1.27)) hide)
@@
     (in_bom yes) (on_board yes) (fields_autoplaced)
     (property "Reference" "SW4" (id 0) (at 119.38 182.88 0))
-    (property "Value" "Backward" (id 1) (at 119.38 185.42 0))
+    (property "Value" "Out" (id 1) (at 119.38 185.42 0))
     (property "Footprint" "Button_Switch_THT:SW_PUSH_6mm" (id 2) (at 119.38 185.42 0)
       (effects (font (size 1.27 1.27)) hide)
@@
     )
     (path "/6220fb82-383d-4273-a0b1-24ac30cce5c6"
-      (reference "SW3") (unit 1) (value "Forward") (footprint "Button_Switch_THT:SW_PUSH_6mm")
+      (reference "SW3") (unit 1) (value "In") (footprint "Button_Switch_THT:SW_PUSH_6mm")
     )
     (path "/8782b0c5-2408-4373-885f-aa7ea3bdfd26"
-      (reference "SW4") (unit 1) (value "Backward") (footprint "Button_Switch_THT:SW_PUSH_6mm")
+      (reference "SW4") (unit 1) (value "Out") (footprint "Button_Switch_THT:SW_PUSH_6mm")
     )
     (path "/3a3d733e-b901-49ad-9f29-c15eaf58f59d"

Commit message: Moved pwm chans to fit pwm hw pairs in RP2040
Connections:
- net Knife: now also U1.22 (GPIO17); no longer U1.27 (GPIO21)
- net Servo_0_LPWM: now also U1.25 (GPIO19); no longer U1.24 (GPIO18)
- net Servo_0_RPWM: now also U1.24 (GPIO18); no longer U1.22 (GPIO17)
- net Servo_1_LPWM: now also U1.27 (GPIO21); no longer U1.26 (GPIO20)
- net Servo_1_RPWM: now also U1.26 (GPIO20); no longer U1.25 (GPIO19)
