File: pcb/StickerCutter.kicad_sch (KiCad schematic)
At the start: 18 parts, among them J1 24V, J3 Line Sensor, J4 Paper Sensor, J5 ENC_0, J6 ENC_1, SW1 F1, SW2 F2, SW3 In, SW4 Out, SW5 Left, SW6 Right, U1 Pico, U2 DC-DC_LM2596s, U3 LCD20x4_HD44780, U4 PWM_MOS_15A

Commit message: Added rotary encoder
Connections:
- net AGND: no longer U1.33 (AGND)
- net Sense Line: no longer U1.32 (GPIO27_ADC1)
- net Sense Paper: no longer U1.31 (GPIO26_ADC0)
- net ROT_ENC_SWITCH: now reaches U1.34 (GPIO28_ADC2)
- new net ROT_ENC_0_B: U1.31 (GPIO26_ADC0), U1.32 (GPIO27_ADC1)
Changed lines of the file:
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@@
+    (stroke (width 0) (type default) (color 0 0 0 0))
+  )
+  (wire (pts (xy 87.63 109.22) (xy 105.41 109.22))
     (stroke (width 0) (type default) (color 0 0 0 0))
   )
@@
   )
   (wire (pts (xy 40.64 104.14) (xy 52.07 104.14))
-    (stroke (width 0) (type default) (color 0 0 0 0))
-  )
-  (wire (pts (xy 87.63 111.76) (xy 103.505 111.76))
     (stroke (width 0) (type default) (color 0 0 0 0))
   )
@@
     (effects (font (size 1.27 1.27)) (justify left bottom))
   )
-  (label "Sense Line" (at 103.505 114.3 180)
+  (label "ROT_ENC_0_B" (at 103.505 114.3 180)
+    (effects (font (size 1.27 1.27)) (justify right bottom))
+  )
+  (label "ROT_ENC_SWITCH" (at 105.41 109.22 180)
     (effects (font (size 1.27 1.27)) (justify right bottom))
   )
@@
     (effects (font (size 1.27 1.27)) (justify left bottom))
   )
-  (label "Sense Paper" (at 103.505 116.84 180)
+  (label "ROT_ENC_0_B" (at 103.505 116.84 180)
     (effects (font (size 1.27 1.27)) (justify right bottom))
   )
@@
     (effects (font (size 1.27 1.27)) (justify right bottom))
   )
-  (label "AGND" (at 103.505 111.76 180)
-    (effects (font (size 1.27 1.27)) (justify right bottom))
-  )
